Commit message: sync https://www.lejuhub.com/highlydynamic/lejulab/commit/0e0ab239a443bf082d8c15f073f93ce497603aba

File: src/leju_assets/models/biped_s46/urdf/drake/biped_v3_arm.urdf (robot description, URDF)
Before this commit: robot biped_v3_arm, 15 links, 14 joints
Links:
- removed link torso
- added link base_link, mass 26.8206; visual mesh filename=../../meshes/torso.STL
- added link zarm_l7_end_effector; collision sphere radius=0.005
- added link zarm_l7_virtual_thumb_link; collision sphere radius=0.005
- added link zarm_r7_end_effector; collision sphere radius=0.005
- added link zarm_r7_virtual_thumb_link; collision sphere radius=0.005
Joints:
- added joint zarm_l7_end_effector_joint: type fixed, parent zarm_l7_link, child zarm_l7_end_effector, origin xyz=0 -0.03 -0.17 rpy=0 0 0
- added joint zarm_l7_virtual_thumb_joint_ee: type fixed, parent zarm_l7_end_effector, child zarm_l7_virtual_thumb_link, origin xyz=0.15 0 0 rpy=0 0 0
- added joint zarm_r7_end_effector_joint: type fixed, parent zarm_r7_link, child zarm_r7_end_effector, origin xyz=0 0.03 -0.17 rpy=0 0 0
- added joint zarm_r7_virtual_thumb_joint_ee: type fixed, parent zarm_r7_end_effector, child zarm_r7_virtual_thumb_link, origin xyz=0.15 0 0 rpy=0 0 0
- joint zarm_l1_joint: limit lower=-3.14159265358979 upper=1.5707963267949 effort=100.0 velocity=41.3433333333333 -> lower=-2.4 upper=0.6 effort=100.0 velocity=41.3433333333333; origin xyz=-0.017499853 0.29269999999999996 0.4245 rpy=0 0 0 -> xyz=-0.017499853 0.29269999999999996 0.445 rpy=0 0 0; parent torso -> base_link
- joint zarm_l2_joint: limit lower=-0.349065850398866 upper=2.0943951023932 effort=50.0 velocity=19.154 -> lower=-0.349065850398866 upper=1.46 effort=50.0 velocity=19.154
- joint zarm_l3_joint: limit lower=-1.5707963267949 upper=1.5707963267949 effort=39.0 velocity=18.84 -> lower=-1.5707963267949 upper=0.46 effort=39.0 velocity=18.84
- joint zarm_l4_joint: limit lower=-2.61799387799149 upper=0.0 effort=50.0 velocity=18.84 -> lower=-2.61799387799149 upper=0.0 effort=50.0 velocity=8.37333333333333; origin xyz=0.0200000000000006 0 -0.283699999999996 rpy=0 0 0 -> xyz=0.0200000000000001 0 -0.2837 rpy=0 0 0
- joint zarm_l5_joint: limit lower=-1.5707963267949 upper=1.5707963267949 effort=12.0 velocity=21.666 -> lower=-1.5707963267949 upper=1.5707963267949 effort=12.0 velocity=7.32666666666667; origin xyz=-0.0200000000000025 0 -0.127037274261591 rpy=0 0 0 -> xyz=-0.02 0 -0.126000000138651 rpy=0 0 0
- joint zarm_l6_joint: limit lower=-1.30899693899575 upper=0.698131700797732 effort=12.0 velocity=21.666 -> lower=-1.30899693899575 upper=0.698131700797732 effort=12.0 velocity=7.32666666666667; origin xyz=0.000199999999999079 0 -0.106462725738415 rpy=0 0 0 -> xyz=0 0 -0.107499999861353 rpy=0 0 0
- joint zarm_l7_joint: limit lower=-0.698131700797732 upper=0.698131700797732 effort=12.0 velocity=21.666 -> lower=-0.698131700797732 upper=0.698131700797732 effort=12.0 velocity=7.32666666666667; origin xyz=0 0 -0.0210004653879916 rpy=0 0 0 -> xyz=0 0 -0.0209999999999992 rpy=0 0 0
- joint zarm_r1_joint: limit lower=-3.14159265358979 upper=1.5707963267949 effort=100.0 velocity=41.3433333333333 -> lower=-2.4 upper=0.6 effort=100.0 velocity=41.3433333333333; origin xyz=-0.017499853 -0.29269999999999996 0.4245 rpy=0 0 0 -> xyz=-0.017499853 -0.29269999999999996 0.445 rpy=0 0 0; parent torso -> base_link
- joint zarm_r2_joint: limit lower=-2.0943951023932 upper=0.349065850398866 effort=50.0 velocity=19.154 -> lower=-1.46 upper=0.349065850398866 effort=50.0 velocity=19.154
- joint zarm_r3_joint: limit lower=-1.5707963267949 upper=1.5707963267949 effort=39.0 velocity=18.84 -> lower=-0.46 upper=1.5707963267949 effort=39.0 velocity=18.84
- joint zarm_r4_joint: limit lower=-2.61799387799149 upper=0.0 effort=50.0 velocity=18.84 -> lower=-2.61799387799149 upper=0.0 effort=50.0 velocity=8.37333333333333; origin xyz=0.0200000000000024 0 -0.2837 rpy=0 0 0 -> xyz=0.0199999999999998 0 -0.2837 rpy=0 0 0
- joint zarm_r5_joint: limit lower=-1.5707963267949 upper=1.5707963267949 effort=12.0 velocity=21.666 -> lower=-1.5707963267949 upper=1.5707963267949 effort=12.0 velocity=7.32666666666667; origin xyz=-0.0200000000000001 0 -0.127037274261587 rpy=0 0 0 -> xyz=-0.0199999999999997 0 -0.126000000138651 rpy=0 0 0
- joint zarm_r6_joint: limit lower=-0.698131700797732 upper=1.30899693899575 effort=12.0 velocity=21.666 -> lower=-0.698131700797732 upper=1.30899693899575 effort=12.0 velocity=7.32666666666667; origin xyz=0 0 -0.106462725738415 rpy=0 0 0 -> xyz=0 0 -0.107499999861352 rpy=0 0 0
- joint zarm_r7_joint: limit lower=-0.698131700797732 upper=0.698131700797732 effort=12.0 velocity=21.666 -> lower=-0.698131700797732 upper=0.698131700797732 effort=12.0 velocity=7.32666666666667; origin xyz=0 0 -0.0209999999999999 rpy=0 0 0 -> xyz=0 0 -0.0210000000000031 rpy=0 0 0

File: src/leju_assets/models/biped_s52/urdf/drake/biped_v3_arm.urdf (robot description, URDF)
Before this commit: robot biped_s52, 18 links, 17 joints
Links:
- added link zarm_l7_virtual_thumb_link; collision sphere radius=0.005
- added link zarm_r7_virtual_thumb_link; collision sphere radius=0.005
- link base_link: mass 6.48663928 -> 7.06405; geometry visual mesh filename=../../meshes/torso.STL
- link waist_yaw_link: mass 18.01415568 -> 20.63616
- link zarm_l1_link: mass 0.91653322 -> 0.94521
- link zarm_l2_link: mass 0.3876739 -> 0.41921
- link zarm_l3_link: mass 1.77926875 -> 1.78857
- link zarm_l4_link: mass 0.58507821 -> 0.63149
- link zarm_l5_link: mass 0.68679955 -> 0.60828
- link zarm_l6_link: mass 0.39387181 -> 0.50616
- link zarm_l7_end_effector: geometry 
- link zarm_l7_link: mass 0.61537779 -> 0.18940
- link zarm_r1_link: mass 0.92062797 -> 0.92947
- link zarm_r2_link: mass 0.38768053 -> 0.41523
- link zarm_r3_link: mass 1.77969208 -> 1.78473
- link zarm_r4_link: mass 0.58514611 -> 0.63548
- link zarm_r5_link: mass 0.68473867 -> 0.61021
- link zarm_r6_link: mass 0.39247462 -> 0.53821
- link zarm_r7_end_effector: geometry 
- link zarm_r7_link: mass 0.61562202 -> 0.19960
Joints:
- added joint zarm_l7_virtual_thumb_joint_ee: type fixed, parent zarm_l7_end_effector, child zarm_l7_virtual_thumb_link, origin xyz=0.15 0 0 rpy=0 0 0
- added joint zarm_r7_virtual_thumb_joint_ee: type fixed, parent zarm_r7_end_effector, child zarm_r7_virtual_thumb_link, origin xyz=0.15 0 0 rpy=0 0 0
- joint waist_yaw_joint: limit lower=-3.14159 upper=3.14159 effort=180.0 velocity=23.55 -> lower=-3.14159 upper=3.14159 effort=102.0 velocity=8.7
- joint zarm_l1_joint: limit lower=-2.4 upper=0.6 effort=100.0 velocity=41.3433333333333 -> lower=-3.14159265358979 upper=1.5707963267949 effort=66.0 velocity=18.8; origin xyz=-0.003 0.2547 0.2831 rpy=0 0 0 -> xyz=-0.003 0.2527 0.283 rpy=0 0 0
- joint zarm_l2_joint: limit lower=-0.349065850398866 upper=1.46 effort=50.0 velocity=19.154 -> lower=-0.349065850398866 upper=3.49065850398866 effort=75.0 velocity=8.0
- joint zarm_l3_joint: limit lower=-1.5707963267949 upper=0.46 effort=39.0 velocity=18.84 -> lower=-1.48352986419518 upper=1.48352986419518 effort=57.0 velocity=7.5; origin xyz=0 0 -0.104 rpy=0 0 0 -> xyz=0 0 0 rpy=0 0 0
- joint zarm_l4_joint: limit lower=-2.61799387799149 upper=0.0 effort=50.0 velocity=18.84 -> lower=-2.61799387799149 upper=0.0 effort=75.0 velocity=8.0; origin xyz=0.02 0 -0.1797 rpy=0 0 0 -> xyz=0.02 0 -0.2837 rpy=0 0 0
- joint zarm_l5_joint: limit lower=-1.5707963267949 upper=1.5707963267949 effort=12.0 velocity=21.666 -> lower=-1.5707963267949 upper=1.5707963267949 effort=14.1 velocity=17.5; origin xyz=-0.02 0 -0.1195 rpy=0 0 0 -> xyz=-0.02 0 -0.1201 rpy=0 0 0
- joint zarm_l6_joint: limit lower=-1.30899693899575 upper=0.698131700797732 effort=12.0 velocity=21.666 -> lower=-1.30899693899575 upper=0.698131700797732 effort=14.1 velocity=17.5; origin xyz=0 0 -0.114 rpy=0 0 0 -> xyz=0.0 0 -0.114 rpy=0 0 0
- joint zarm_l7_end_effector_joint: origin xyz=0 -0.03 -0.17 rpy=0 0 0 -> xyz=0 0.0 -0.17 rpy=0 0 0
- joint zarm_l7_joint: limit lower=-0.698131700797732 upper=0.698131700797732 effort=12.0 velocity=21.666 -> lower=-0.698131700797732 upper=0.698131700797732 effort=14.1 velocity=17.5; origin xyz=-0.0002 0 -0.021 rpy=0 0 0 -> xyz=0 0 -0.021 rpy=0 0 0
- joint zarm_r1_joint: limit lower=-2.4 upper=0.6 effort=100.0 velocity=41.3433333333333 -> lower=-3.14159265358979 upper=1.5707963267949 effort=66.0 velocity=18.8; origin xyz=-0.003 -0.2547 0.2831 rpy=0 0 0 -> xyz=-0.003 -0.2527 0.283 rpy=0 0 0
- joint zarm_r2_joint: limit lower=-1.46 upper=0.349065850398866 effort=50.0 velocity=19.154 -> lower=-3.49065850398866 upper=0.349065850398866 effort=75.0 velocity=8.0
- joint zarm_r3_joint: limit lower=-0.46 upper=1.5707963267949 effort=39.0 velocity=18.84 -> lower=-1.48352986419518 upper=1.48352986419518 effort=57.0 velocity=7.5; origin xyz=0 0 -0.104 rpy=0 0 0 -> xyz=0 0 0 rpy=0 0 0
- joint zarm_r4_joint: limit lower=-2.61799387799149 upper=0.0 effort=50.0 velocity=18.84 -> lower=-2.61799387799149 upper=0.0 effort=75.0 velocity=8.0; origin xyz=0.02 0 -0.1797 rpy=0 0 0 -> xyz=0.02 0 -0.2837 rpy=0 0 0
- joint zarm_r5_joint: limit lower=-1.5707963267949 upper=1.5707963267949 effort=12.0 velocity=21.666 -> lower=-1.5707963267949 upper=1.5707963267949 effort=14.1 velocity=17.5; origin xyz=-0.02 0 -0.1195 rpy=0 0 0 -> xyz=-0.02 0 -0.1201 rpy=0 0 0
- joint zarm_r6_joint: limit lower=-0.698131700797732 upper=1.30899693899575 effort=12.0 velocity=21.666 -> lower=-0.698131700797732 upper=1.30899693899575 effort=14.1 velocity=17.5; origin xyz=0 0 -0.114 rpy=0 0 0 -> xyz=0.0 0 -0.114 rpy=0 0 0
- joint zarm_r7_end_effector_joint: origin xyz=0 0.03 -0.17 rpy=0 0 0 -> xyz=0 0.0 -0.17 rpy=0 0 0
- joint zarm_r7_joint: limit lower=-0.698131700797732 upper=0.698131700797732 effort=12.0 velocity=21.666 -> lower=-0.698131700797732 upper=0.698131700797732 effort=14.1 velocity=17.5; origin xyz=0 0 -0.022284 rpy=0 0 0 -> xyz=0.0 0 -0.021 rpy=0 0 0
