Commit message: sync https://www.lejuhub.com/highlydynamic/lejulab/commit/fe213f8aac422dd1877b756b5fe1d4e54ef00ade

File: src/leju_assets/models/biped_s17/urdf/biped_s17.urdf (robot description, URDF)
Before this commit: robot biped_s17, 39 links, 38 joints
Links:
- removed link waist_yaw_link
- added link camera_base, mass 0.00001000; visual mesh filename=package://kuavo_assets/models/biped_s17/meshes/head_camera_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
- added link head_radar, mass 0.00000100; visual mesh filename=package://kuavo_assets/models/biped_s17/meshes/head_radar.S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
- added link l_handball, mass 0.17660000; visual mesh filename=package://kuavo_assets/models/biped_s17/meshes/l_handball.S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
- added link r_handball, mass 0.17660000; visual mesh filename=package://kuavo_assets/models/biped_s17/meshes/r_handball.S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
- added link torso, mass 8.37744703; collision box size=0.14 0.2 0.26; collision cylinder length=0.125 radius=0.008
- link base_link: mass 4.853 -> 5.27737344; geometry collision sphere radius=0.08; visual mesh filename=package://kuavo_assets/models/biped_s17/meshes/waist.STL
- link leg_l1_link: mass 0.62568928 -> 0.6865; geometry collision capsule length=0.06 radius=0.042; collision capsule length=0.06 radius=0.042
- link leg_l2_link: mass 2.03159924 -> 2.054; geometry collision capsule length=0.14 radius=0.055; visual mesh filename=package://kuavo_assets/models/biped_s17/meshes/l_leg_roll.S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
- link leg_l3_link: mass 3.38846623 -> 3.2746; geometry collision capsule length=0.03 radius=0.055; visual mesh filename=package://kuavo_assets/models/biped_s17/meshes/l_leg_yaw.STL
- link leg_l4_link: mass 2.61852 -> 2.4454; geometry collision capsule length=0.05 radius=0.005; collision capsule length=0.05 radius=0.005
- link leg_l5_link: mass 0.10854305 -> 0.1314; geometry visual mesh filename=package://kuavo_assets/models/biped_s17/meshes/l_foot_pitch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
- link leg_l6_link: mass 0.43610846 -> 0.5783271; geometry collision box size=0.12 0.07 0.01; collision cylinder length=0.01 radius=0.035
- link leg_r1_link: mass 0.62568928 -> 0.6865; geometry collision capsule length=0.06 radius=0.042; collision capsule length=0.06 radius=0.042
- link leg_r2_link: mass 2.03159924 -> 2.054; geometry collision capsule length=0.14 radius=0.055; visual mesh filename=package://kuavo_assets/models/biped_s17/meshes/r_leg_roll.S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
- link leg_r3_link: mass 3.38846623 -> 3.2746; geometry collision capsule length=0.03 radius=0.055; visual mesh filename=package://kuavo_assets/models/biped_s17/meshes/r_leg_yaw.STL
- link leg_r4_link: mass 2.61852 -> 2.4454; geometry collision capsule length=0.05 radius=0.005; collision capsule length=0.05 radius=0.005
- link leg_r5_link: mass 0.10854305 -> 0.1314; geometry visual mesh filename=package://kuavo_assets/models/biped_s17/meshes/r_foot_pitch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
- link leg_r6_link: mass 0.43610846 -> 0.5783271; geometry collision box size=0.12 0.07 0.01; collision cylinder length=0.01 radius=0.035
- link zarm_l1_link: mass 0.80328906 -> 0.84760000; geometry collision capsule length=0.04 radius=0.04; visual mesh filename=package://kuavo_assets/models/biped_s17/meshes/l_arm_pitch.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
- link zarm_l2_link: mass 0.32360735 -> 0.36680000; geometry collision capsule length=0.035 radius=0.035; visual mesh filename=package://kuavo_assets/models/biped_s17/meshes/l_arm_roll.S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
- link zarm_l3_link: mass 1.46578996 -> 1.51660000; geometry collision capsule length=0.05 radius=0.035; visual mesh filename=package://kuavo_assets/models/biped_s17/meshes/l_arm_yaw.STL
- link zarm_l4_link: mass 0.42136972 -> 0.34500000; geometry collision capsule length=0.03 radius=0.045; collision capsule length=0.12 radius=0.02
- link zarm_r1_link: mass 0.80328906 -> 0.84760000; geometry collision capsule length=0.04 radius=0.04; visual mesh filename=package://kuavo_assets/models/biped_s17/meshes/r_arm_pitch.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
- link zarm_r2_link: mass 0.32360735 -> 0.36680000; geometry collision capsule length=0.035 radius=0.035; visual mesh filename=package://kuavo_assets/models/biped_s17/meshes/r_arm_roll.S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
- link zarm_r3_link: mass 1.46578996 -> 1.51660000; geometry collision capsule length=0.05 radius=0.035; visual mesh filename=package://kuavo_assets/models/biped_s17/meshes/r_arm_yaw.STL
- link zarm_r4_link: mass 0.42136972 -> 0.34500000; geometry collision capsule length=0.03 radius=0.045; collision capsule length=0.12 radius=0.02
- link zhead_1_link: mass 1.03077542 -> 1.07555742; geometry collision capsule length=0.1 radius=0.035; visual mesh filename=package://kuavo_assets/models/biped_s17/meshes/head_yaw.STL
- link zhead_2_link: mass 0.33654975 -> 0.61000000; geometry collision sphere radius=0.075; visual mesh filename=package://kuavo_assets/models/biped_s17/meshes/head_pitch.S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
Joints:
- added joint camera_base_joint: type fixed, parent zhead_2_link, child camera_base, origin xyz=0.047118 0 0.051192 rpy=0 0.27152 0
- added joint head_radar_joint: type fixed, parent zhead_1_link, child head_radar, origin xyz=0 0 -0.026453 rpy=0 0 0
- added joint l_handball_joint: type fixed, parent zarm_l4_link, child l_handball, origin xyz=0 0 -0.085236 rpy=0 0 0
- added joint r_handball_joint: type fixed, parent zarm_r4_link, child r_handball, origin xyz=0 0 -0.085236 rpy=0 0 0
- joint leg_l1_joint: origin xyz=0.0 0.12441237 -0.22115341 rpy=0 0 0 -> xyz=0 0.12441 -0.22265 rpy=0 0 0
- joint leg_r1_joint: origin xyz=0.0 -0.12441237 -0.22115341 rpy=0 0 0 -> xyz=0.0 -0.12441 -0.22265 rpy=0 0 0
- joint waist_yaw_joint: child waist_yaw_link -> torso
- joint zarm_l1_joint: origin xyz=0.0 0.18100293 0.23992606 rpy=0 0 0 -> xyz=0 0.181 0.23843 rpy=0 0 0; parent waist_yaw_link -> torso
- joint zarm_l4_joint: origin xyz=0 0.0 -0.20533 rpy=0 0 0 -> xyz=0 0 -0.2085 rpy=0 0 0
- joint zarm_r1_joint: origin xyz=0.0 -0.18100293 0.23992606 rpy=0 0 0 -> xyz=0 -0.181 0.23843 rpy=0 0 0; parent waist_yaw_link -> torso
- joint zarm_r4_joint: origin xyz=0 -0.0 -0.20533 rpy=0 0 0 -> xyz=0 0 -0.2085 rpy=0 0 0
- joint zhead_1_joint: origin xyz=0.004 0 0.35618 rpy=0 0 0 -> xyz=0.0042 0 0.35369 rpy=0 0 0; parent waist_yaw_link -> torso

File: src/leju_assets/models/biped_s17/urdf/biped_s17_gazebo.urdf (robot description, URDF)
Before this commit: robot biped_s17, 39 links, 38 joints
Links:
- removed link waist_yaw_link
- added link camera_base, mass 0.00001000; visual mesh filename=package://kuavo_assets/models/biped_s17/meshes/head_camera_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
- added link head_radar, mass 0.00000100; visual mesh filename=package://kuavo_assets/models/biped_s17/meshes/head_radar.S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
- added link l_handball, mass 0.17660000; visual mesh filename=package://kuavo_assets/models/biped_s17/meshes/l_handball.S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
- added link r_handball, mass 0.17660000; visual mesh filename=package://kuavo_assets/models/biped_s17/meshes/r_handball.S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
- added link torso, mass 8.37744703; collision box size=0.14 0.2 0.26; collision cylinder length=0.013 radius=0.005
- link base_link: mass 4.8567 -> 5.27737344; geometry collision box size=0.14 0.2 0.26; collision cylinder length=0.125 radius=0.008
- link leg_l1_link: mass 0.62568928 -> 0.6865; geometry visual mesh filename=package://kuavo_assets/models/biped_s17/meshes/l_leg_pitch.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
- link leg_l2_link: mass 2.03159924 -> 2.054; geometry visual mesh filename=package://kuavo_assets/models/biped_s17/meshes/l_leg_roll.S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
- link leg_l3_link: mass 3.38846623 -> 3.2746; geometry visual mesh filename=package://kuavo_assets/models/biped_s17/meshes/l_leg_yaw.STL
- link leg_l4_link: mass 2.61852 -> 2.4454; geometry visual mesh filename=package://kuavo_assets/models/biped_s17/meshes/l_knee.STL
- link leg_l5_link: mass 0.10854305 -> 0.1314; geometry visual mesh filename=package://kuavo_assets/models/biped_s17/meshes/l_foot_pitch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
- link leg_l6_link: mass 0.43610846 -> 0.5783271; geometry visual mesh filename=package://kuavo_assets/models/biped_s17/meshes/l_foot_roll.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
- link leg_r1_link: mass 0.62568928 -> 0.6865; geometry visual mesh filename=package://kuavo_assets/models/biped_s17/meshes/r_leg_pitch.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
- link leg_r2_link: mass 2.03159924 -> 2.054; geometry visual mesh filename=package://kuavo_assets/models/biped_s17/meshes/r_leg_roll.S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
- link leg_r3_link: mass 3.38846623 -> 3.2746; geometry visual mesh filename=package://kuavo_assets/models/biped_s17/meshes/r_leg_yaw.STL
- link leg_r4_link: mass 2.61852 -> 2.4454; geometry visual mesh filename=package://kuavo_assets/models/biped_s17/meshes/r_knee.STL
- link leg_r5_link: mass 0.10854305 -> 0.1314; geometry visual mesh filename=package://kuavo_assets/models/biped_s17/meshes/r_foot_pitch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
- link leg_r6_link: mass 0.43610846 -> 0.5783271; geometry visual mesh filename=package://kuavo_assets/models/biped_s17/meshes/r_foot_roll.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
- link zarm_l1_link: mass 0.80328906 -> 0.84760000; geometry visual mesh filename=package://kuavo_assets/models/biped_s17/meshes/l_arm_pitch.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
- link zarm_l2_link: mass 0.32360735 -> 0.36680000; geometry visual mesh filename=package://kuavo_assets/models/biped_s17/meshes/l_arm_roll.S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
- link zarm_l3_link: mass 1.46578996 -> 1.51660000; geometry visual mesh filename=package://kuavo_assets/models/biped_s17/meshes/l_arm_yaw.STL
- link zarm_l4_link: mass 0.42136972 -> 0.34500000; geometry visual mesh filename=package://kuavo_assets/models/biped_s17/meshes/l_forearm.STL
- link zarm_r1_link: mass 0.80328906 -> 0.84760000; geometry visual mesh filename=package://kuavo_assets/models/biped_s17/meshes/r_arm_pitch.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
- link zarm_r2_link: mass 0.32360735 -> 0.36680000; geometry visual mesh filename=package://kuavo_assets/models/biped_s17/meshes/r_arm_roll.S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
- link zarm_r3_link: mass 1.46578996 -> 1.51660000; geometry visual mesh filename=package://kuavo_assets/models/biped_s17/meshes/r_arm_yaw.STL
- link zarm_r4_link: mass 0.42136972 -> 0.34500000; geometry visual mesh filename=package://kuavo_assets/models/biped_s17/meshes/r_forearm.STL
- link zhead_1_link: mass 1.03077542 -> 1.07555742; geometry visual mesh filename=package://kuavo_assets/models/biped_s17/meshes/head_yaw.STL
- link zhead_2_link: mass 0.33654975 -> 0.61000000; geometry collision sphere radius=0.075; visual mesh filename=package://kuavo_assets/models/biped_s17/meshes/head_pitch.S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
Joints:
- added joint camera_base_joint: type fixed, parent zhead_2_link, child camera_base, origin xyz=0.047118 0 0.051192 rpy=0 0.27152 0
- added joint head_radar_joint: type fixed, parent zhead_1_link, child head_radar, origin xyz=0 0 -0.026453 rpy=0 0 0
- added joint l_handball_joint: type fixed, parent zarm_l4_link, child l_handball, origin xyz=0 0 -0.085236 rpy=0 0 0
- added joint r_handball_joint: type fixed, parent zarm_r4_link, child r_handball, origin xyz=0 0 -0.085236 rpy=0 0 0
- joint leg_l1_joint: origin xyz=0.0 0.12441237 -0.22115341 rpy=0 0 0 -> xyz=0 0.12441 -0.22265 rpy=0 0 0
- joint leg_l5_joint: limit lower=-0.872664625997165 upper=0.523598775598299 effort=37 velocity=17.0 -> lower=-0.872664625997165 upper=0.523598775598299 effort=74 velocity=17.0
- joint leg_l6_joint: limit lower=-0.261799387799149 upper=0.261799387799149 effort=37 velocity=17.0 -> lower=-0.261799387799149 upper=0.261799387799149 effort=74 velocity=17.0
- joint leg_r1_joint: origin xyz=0.0 -0.12441237 -0.22115341 rpy=0 0 0 -> xyz=0.0 -0.12441 -0.22265 rpy=0 0 0
- joint leg_r5_joint: limit lower=-0.872664625997165 upper=0.523598775598299 effort=37 velocity=17.0 -> lower=-0.872664625997165 upper=0.523598775598299 effort=74 velocity=17.0
- joint leg_r6_joint: limit lower=-0.261799387799149 upper=0.261799387799149 effort=37 velocity=17.0 -> lower=-0.261799387799149 upper=0.261799387799149 effort=74 velocity=17.0
- joint waist_yaw_joint: child waist_yaw_link -> torso
- joint zarm_l1_joint: origin xyz=0.0 0.18100293 0.23992606 rpy=0 0 0 -> xyz=0 0.181 0.23843 rpy=0 0 0; parent waist_yaw_link -> torso
- joint zarm_l4_joint: origin xyz=0 0.0 -0.20533 rpy=0 0 0 -> xyz=0 0 -0.2085 rpy=0 0 0
- joint zarm_r1_joint: origin xyz=0.0 -0.18100293 0.23992606 rpy=0 0 0 -> xyz=0 -0.181 0.23843 rpy=0 0 0; parent waist_yaw_link -> torso
- joint zarm_r4_joint: origin xyz=0 -0.0 -0.20533 rpy=0 0 0 -> xyz=0 0 -0.2085 rpy=0 0 0
- joint zhead_1_joint: origin xyz=0.004 0 0.35618 rpy=0 0 0 -> xyz=0.0042 0 0.35369 rpy=0 0 0; parent waist_yaw_link -> torso

File: src/leju_assets/models/biped_s17/urdf/biped_s17_gazebo.xacro (robot description, xacro)
@@ -2,5 +2,5 @@
 <robot xmlns:xacro="http://ros.org/wiki/xacro" name="biped_s17_with_realsense">
   <!-- 引入机器人主体 -->
-  <xacro:include filename="$(find leju_assets)/models/biped_s17/urdf/biped_s17_gazebo.urdf"/>
+  <xacro:include filename="$(find kuavo_assets)/models/biped_s17/urdf/biped_s17_gazebo.urdf"/>
   <!-- depth cam 设置 -->
   <xacro:include filename="$(find realsense_ros_gazebo)/xacro/depthcam.xacro"/>

File: src/leju_assets/models/biped_s17/urdf/drake/biped_v3.urdf (robot description, URDF)
Before this commit: robot biped_v3, 14 links, 13 joints
Links:
- link leg_l1_link: mass 0.62568928 -> 0.6865
- link leg_l2_link: mass 2.03159924 -> 2.054
- link leg_l3_link: mass 3.38846623 -> 3.2746
- link leg_l4_link: mass 2.61852 -> 2.4454
- link leg_l5_link: mass 0.10854305 -> 0.1314
- link leg_l6_link: mass 0.43610846 -> 0.5783271
- link leg_r1_link: mass 0.62568928 -> 0.6865
- link leg_r2_link: mass 2.03159924 -> 2.054
- link leg_r3_link: mass 3.38846623 -> 3.2746
- link leg_r4_link: mass 2.61852 -> 2.4454
- link leg_r5_link: mass 0.10854305 -> 0.1314
- link leg_r6_link: mass 0.43610846 -> 0.5783271
- link torso: mass 18.2491 -> 15.78214703
- link waist: mass 4.853 -> 5.27737344
Joints:
- joint leg_l1_joint: limit lower=-3.228 upper=2.44346 effort=180 velocity=23.55 -> lower=-3.228 upper=2.44346 effort=150 velocity=14.6; origin xyz=0.0 0.12441237 -0.22115341 rpy=0 0 0 -> xyz=0 0.12441 -0.22265 rpy=0 0 0
- joint leg_l2_joint: limit lower=-0.837758 upper=2.40855 effort=100 velocity=41.3433333333333 -> lower=-0.837758 upper=2.40855 effort=150 velocity=14.6
- joint leg_l3_joint: limit lower=-1.7453 upper=1.7453 effort=100 velocity=41.3433333333333 -> lower=-1.7453 upper=1.7453 effort=70 velocity=12.0
- joint leg_l4_joint: limit lower=-0.08726646 upper=2.530727 effort=180 velocity=23.55 -> lower=-0.08726646 upper=2.530727 effort=150 velocity=14.6
- joint leg_l5_joint: limit lower=-0.872664625997165 upper=0.523598775598299 effort=36.0 velocity=23.0266666666667 -> lower=-0.872664625997165 upper=0.523598775598299 effort=74 velocity=17.0
- joint leg_l6_joint: limit lower=-0.261799387799149 upper=0.261799387799149 effort=36 velocity=23.0266666666667 -> lower=-0.261799387799149 upper=0.261799387799149 effort=74 velocity=17.0
- joint leg_r1_joint: limit lower=-3.228 upper=2.44346 effort=180 velocity=23.55 -> lower=-2.44346 upper=3.228 effort=150 velocity=14.6; origin xyz=0.0 -0.12441237 -0.22115341 rpy=0 0 0 -> xyz=0.0 -0.12441 -0.22265 rpy=0 0 0
- joint leg_r2_joint: limit lower=-2.40855 upper=0.837758 effort=100 velocity=41.3433333333333 -> lower=-2.40855 upper=0.837758 effort=150 velocity=14.6
- joint leg_r3_joint: limit lower=-1.7453 upper=1.7453 effort=100 velocity=41.3433333333333 -> lower=-1.7453 upper=1.7453 effort=70 velocity=12.0
- joint leg_r4_joint: limit lower=-0.08726646 upper=2.530727 effort=180 velocity=23.55 -> lower=-0.08726646 upper=2.530727 effort=150 velocity=14.6
- joint leg_r5_joint: limit lower=-0.872664625997165 upper=0.523598775598299 effort=36.0 velocity=23.0266666666667 -> lower=-0.872664625997165 upper=0.523598775598299 effort=74 velocity=17.0
- joint leg_r6_joint: limit lower=-0.261799387799149 upper=0.261799387799149 effort=36 velocity=23.0266666666667 -> lower=-0.261799387799149 upper=0.261799387799149 effort=74 velocity=17.0

File: src/leju_assets/models/biped_s17/urdf/drake/biped_v3_all_joint.urdf (robot description, URDF)
Before this commit: robot biped_v3_all_joint, 30 links, 25 joints
Links:
- link leg_l1_link: mass 0.62568928 -> 0.6865
- link leg_l2_link: mass 2.03159924 -> 2.054
- link leg_l3_link: mass 3.38846623 -> 3.2746
- link leg_l4_link: mass 2.61852 -> 2.4454
- link leg_l5_link: mass 0.10854305 -> 0.1314
- link leg_l6_link: mass 0.43610846 -> 0.5783271
- link leg_r1_link: mass 0.62568928 -> 0.6865
- link leg_r2_link: mass 2.03159924 -> 2.054
- link leg_r3_link: mass 3.38846623 -> 3.2746
- link leg_r4_link: mass 2.61852 -> 2.4454
- link leg_r5_link: mass 0.10854305 -> 0.1314
- link leg_r6_link: mass 0.43610846 -> 0.5783271
- link torso: mass 11.5782 -> 8.98734703
- link waist: mass 4.853 -> 5.27737344
- link zarm_l1_link: mass 0.80328906 -> 0.84760000
- link zarm_l2_link: mass 0.32360735 -> 0.36680000
- link zarm_l3_link: mass 1.46578996 -> 1.51660000
- link zarm_l4_link: mass 0.42136972 -> 0.34500000
- link zarm_r1_link: mass 0.80328906 -> 0.84760000
- link zarm_r2_link: mass 0.32360735 -> 0.36680000
- link zarm_r3_link: mass 1.46578996 -> 1.51660000
- link zarm_r4_link: mass 0.42136972 -> 0.34500000
Joints:
- joint leg_l1_joint: limit lower=-3.228 upper=2.44346 effort=180 velocity=23.55 -> lower=-3.228 upper=2.44346 effort=150 velocity=14.6; origin xyz=0.0 0.12441237 -0.22115341 rpy=0 0 0 -> xyz=0 0.12441 -0.22265 rpy=0 0 0
- joint leg_l2_joint: limit lower=-0.837758 upper=2.40855 effort=100 velocity=41.3433333333333 -> lower=-0.837758 upper=2.40855 effort=150 velocity=14.6
- joint leg_l3_joint: limit lower=-1.7453 upper=1.7453 effort=100 velocity=41.3433333333333 -> lower=-1.7453 upper=1.7453 effort=70 velocity=12.0
- joint leg_l4_joint: limit lower=-0.08726646 upper=2.530727 effort=180 velocity=23.55 -> lower=-0.08726646 upper=2.530727 effort=150 velocity=14.6
- joint leg_l5_joint: limit lower=-0.872664625997165 upper=0.523598775598299 effort=36 velocity=23.0266666666667 -> lower=-0.872664625997165 upper=0.523598775598299 effort=74 velocity=17.0
- joint leg_l6_joint: limit lower=-0.261799387799149 upper=0.261799387799149 effort=36 velocity=23.0266666666667 -> lower=-0.261799387799149 upper=0.261799387799149 effort=74 velocity=17.0
- joint leg_r1_joint: limit lower=-3.228 upper=2.44346 effort=180 velocity=23.55 -> lower=-2.44346 upper=3.228 effort=150 velocity=14.6; origin xyz=0.0 -0.12441237 -0.22115341 rpy=0 0 0 -> xyz=0.0 -0.12441 -0.22265 rpy=0 0 0
- joint leg_r2_joint: limit lower=-2.40855 upper=0.837758 effort=100 velocity=41.3433333333333 -> lower=-2.40855 upper=0.837758 effort=150 velocity=14.6
- joint leg_r3_joint: limit lower=-1.7453 upper=1.7453 effort=100 velocity=41.3433333333333 -> lower=-1.7453 upper=1.7453 effort=70 velocity=12.0
- joint leg_r4_joint: limit lower=-0.08726646 upper=2.530727 effort=180 velocity=23.55 -> lower=-0.08726646 upper=2.530727 effort=150 velocity=14.6
- joint leg_r5_joint: limit lower=-0.872664625997165 upper=0.523598775598299 effort=36 velocity=23.0266666666667 -> lower=-0.872664625997165 upper=0.523598775598299 effort=74 velocity=17.0
- joint leg_r6_joint: limit lower=-0.261799387799149 upper=0.261799387799149 effort=36 velocity=23.0266666666667 -> lower=-0.261799387799149 upper=0.261799387799149 effort=74 velocity=17.0
- joint zarm_l1_joint: limit lower=-3.14159265358979 upper=2.0943951023932 effort=12 velocity=7.32666666666667 -> lower=-3.14159265358979 upper=2.0943951023932 effort=14.1 velocity=10.5; origin xyz=0.0 0.18100293 0.23992606 rpy=0 0 0 -> xyz=0 0.181 0.23843 rpy=0 0 0
- joint zarm_l2_joint: limit lower=-3.3161 upper=0.52 effort=12 velocity=7.32666666666667 -> lower=-0.52 upper=3.316 effort=37 velocity=15.0
- joint zarm_l3_joint: limit lower=-1.5707963267949 upper=1.5707963267949 effort=12 velocity=7.32666666666667 -> lower=-1.5707963267949 upper=1.5707963267949 effort=37 velocity=15.0
- joint zarm_l4_joint: limit lower=-2.26892802759263 upper=0.08726 effort=12 velocity=7.32666666666667 -> lower=-2.26892802759263 upper=0.08726 effort=37 velocity=15.0; origin xyz=0 0.0 -0.20533 rpy=0 0 0 -> xyz=0 0 -0.2085 rpy=0 0 0
- joint zarm_r1_joint: limit lower=-3.14159265358979 upper=2.0943951023932 effort=12 velocity=7.32666666666667 -> lower=-3.14159265358979 upper=2.0943951023932 effort=14.1 velocity=10.5; origin xyz=0.0 -0.18100293 0.23992606 rpy=0 0 0 -> xyz=0 -0.181 0.23843 rpy=0 0 0
- joint zarm_r2_joint: limit lower=-3.3161 upper=0.52 effort=12 velocity=7.32666666666667 -> lower=-3.3161 upper=0.52 effort=37.0 velocity=15.0
- joint zarm_r3_joint: limit lower=-1.5707963267949 upper=1.5707963267949 effort=12 velocity=7.32666666666667 -> lower=-1.5707963267949 upper=1.5707963267949 effort=37.0 velocity=15.0
- joint zarm_r4_joint: limit lower=-2.26892802759263 upper=0.08726 effort=12 velocity=7.32666666666667 -> lower=-2.26892802759263 upper=0.08726 effort=37.0 velocity=15.0; origin xyz=0 -0.0 -0.20533 rpy=0 0 0 -> xyz=0 0 -0.2085 rpy=0 0 0

File: src/leju_assets/models/biped_s17/urdf/drake/biped_v3_arm.urdf (robot description, URDF)
Before this commit: robot biped_v3_arm, 12 links, 11 joints
Links:
- added link l_handball, mass 0.17660000; visual mesh filename=package://biped_s17/meshes/l_handball.STL
- added link r_handball, mass 0.17660000; visual mesh filename=package://biped_s17/meshes/r_handball.STL
- link torso: mass 8.730 -> 8.37744703
- link waist: mass 4.853 -> 5.27737344
- link zarm_l1_link: mass 0.80328906 -> 0.84760000
- link zarm_l2_link: mass 0.32360735 -> 0.36680000
- link zarm_l3_link: mass 1.46578996 -> 1.51660000
- link zarm_l4_link: mass 0.42136972 -> 0.34500000
- link zarm_r1_link: mass 0.80328906 -> 0.84760000
- link zarm_r2_link: mass 0.32360735 -> 0.36680000
- link zarm_r3_link: mass 1.46578996 -> 1.51660000
- link zarm_r4_link: mass 0.42136972 -> 0.34500000
Joints:
- added joint l_handball_joint: type fixed, parent zarm_l4_link, child l_handball, origin xyz=0 0 -0.085236 rpy=0 0 0
- added joint r_handball_joint: type fixed, parent zarm_r4_link, child r_handball, origin xyz=0 0 -0.085236 rpy=0 0 0
- joint waist: limit lower=-2.0943951023932 upper=2.0943951023932 effort=36.0 velocity=23.0266666666667 -> lower=-2.61799387799149 upper=2.61799387799149 effort=80 velocity=12.0
- joint zarm_l1_joint: origin xyz=0.0 0.18100293 0.23992606 rpy=0 0 0 -> xyz=0 0.181 0.23843 rpy=0 0 0
- joint zarm_l4_joint: origin xyz=0 0.0 -0.20533 rpy=0 0 0 -> xyz=0 0 -0.2085 rpy=0 0 0
- joint zarm_r1_joint: origin xyz=0.0 -0.18100293 0.23992606 rpy=0 0 0 -> xyz=0 -0.181 0.23843 rpy=0 0 0
- joint zarm_r4_joint: origin xyz=0 -0.0 -0.20533 rpy=0 0 0 -> xyz=0 0 -0.2085 rpy=0 0 0
