Commit message: sync https://www.lejuhub.com/highlydynamic/lejulab/commit/fe213f8aac422dd1877b756b5fe1d4e54ef00ade

File: src/leju_assets/models/biped_s17/urdf/drake/biped_v3_full.urdf (robot description, URDF)
Before this commit: robot biped_v3_full, 22 links, 21 joints
Links:
- link leg_l1_link: mass 0.62568928 -> 0.6865
- link leg_l2_link: mass 2.03159924 -> 2.054
- link leg_l3_link: mass 3.38846623 -> 3.2746
- link leg_l4_link: mass 2.61852 -> 2.4454
- link leg_l5_link: mass 0.10854305 -> 0.1314
- link leg_l6_link: mass 0.43610846 -> 0.5783271
- link leg_r1_link: mass 0.42877618 -> 0.6865
- link leg_r2_link: mass 2.4999594 -> 2.054
- link leg_r3_link: mass 3.38846623 -> 3.2746
- link leg_r4_link: mass 2.61852 -> 2.4454
- link leg_r5_link: mass 0.10854305 -> 0.1314
- link leg_r6_link: mass 0.43610846 -> 0.5783271
- link torso: mass 11.9496 -> 9.63014703
- link waist: mass 4.853 -> 5.27737344
- link zarm_l1_link: mass 0.80328906 -> 0.84760000
- link zarm_l2_link: mass 0.32360735 -> 0.36680000
- link zarm_l3_link: mass 1.46578996 -> 1.51660000
- link zarm_l4_link: mass 0.42136972 -> 0.34500000
- link zarm_r1_link: mass 0.80328906 -> 0.84760000
- link zarm_r2_link: mass 0.32360735 -> 0.36680000
- link zarm_r3_link: mass 1.46578996 -> 1.51660000
- link zarm_r4_link: mass 0.42136972 -> 0.34500000
Joints:
- joint leg_l1_joint: limit lower=-3.228 upper=2.44346 effort=180 velocity=23.55 -> lower=-3.228 upper=2.44346 effort=150 velocity=14.6; origin xyz=0.0 0.12441237 -0.22115341 rpy=0 0 0 -> xyz=0 0.12441 -0.22265 rpy=0 0 0
- joint leg_l2_joint: limit lower=-0.837758 upper=2.40855 effort=100 velocity=41.3433333333333 -> lower=-0.837758 upper=2.40855 effort=150 velocity=14.6
- joint leg_l3_joint: limit lower=-1.7453 upper=1.7453 effort=100 velocity=41.3433333333333 -> lower=-1.7453 upper=1.7453 effort=70 velocity=12.0
- joint leg_l4_joint: limit lower=-0.08726646 upper=2.530727 effort=180 velocity=23.55 -> lower=-0.08726646 upper=2.530727 effort=150 velocity=14.6
- joint leg_l5_joint: limit lower=-0.872664625997165 upper=0.523598775598299 effort=36.0 velocity=23.0266666666667 -> lower=-0.872664625997165 upper=0.523598775598299 effort=74 velocity=17.0
- joint leg_l6_joint: limit lower=-0.261799387799149 upper=0.261799387799149 effort=36 velocity=23.0266666666667 -> lower=-0.261799387799149 upper=0.261799387799149 effort=74 velocity=17.0
- joint leg_r1_joint: limit lower=-3.228 upper=2.44346 effort=180 velocity=23.55 -> lower=-2.44346 upper=3.228 effort=150 velocity=14.6; origin xyz=0.0 -0.12441237 -0.22115341 rpy=0 0 0 -> xyz=0.0 -0.12441 -0.22265 rpy=0 0 0
- joint leg_r2_joint: limit lower=-2.40855 upper=0.837758 effort=100 velocity=41.3433333333333 -> lower=-2.40855 upper=0.837758 effort=150 velocity=14.6
- joint leg_r3_joint: limit lower=-1.7453 upper=1.7453 effort=100 velocity=41.3433333333333 -> lower=-1.7453 upper=1.7453 effort=70 velocity=12.0
- joint leg_r4_joint: limit lower=-0.08726646 upper=2.530727 effort=180 velocity=23.55 -> lower=-0.08726646 upper=2.530727 effort=150 velocity=14.6
- joint leg_r5_joint: limit lower=-0.872664625997165 upper=0.523598775598299 effort=36.0 velocity=23.0266666666667 -> lower=-0.872664625997165 upper=0.523598775598299 effort=74 velocity=17.0
- joint leg_r6_joint: limit lower=-0.261799387799149 upper=0.261799387799149 effort=36 velocity=23.0266666666667 -> lower=-0.261799387799149 upper=0.261799387799149 effort=74 velocity=17.0
- joint zarm_l1_joint: limit lower=-3.14159265358979 upper=2.0943951023932 effort=12 velocity=7.32666666666667 -> lower=-3.14159265358979 upper=2.0943951023932 effort=14.1 velocity=10.5; origin xyz=0.0 0.18100293 0.23992606 rpy=0 0 0 -> xyz=0 0.181 0.23843 rpy=0 0 0
- joint zarm_l2_joint: limit lower=-0.52 upper=3.316 effort=12 velocity=7.32666666666667 -> lower=-0.52 upper=3.316 effort=37 velocity=15.0
- joint zarm_l3_joint: limit lower=-1.5707963267949 upper=1.5707963267949 effort=12 velocity=7.32666666666667 -> lower=-1.5707963267949 upper=1.5707963267949 effort=37 velocity=15.0
- joint zarm_l4_joint: limit lower=-2.26892802759263 upper=0.08726 effort=12 velocity=7.32666666666667 -> lower=-2.26892802759263 upper=0.08726 effort=37 velocity=15.0; origin xyz=0 0.0 -0.20533 rpy=0 0 0 -> xyz=0 0 -0.2085 rpy=0 0 0
- joint zarm_r1_joint: limit lower=-3.14159265358979 upper=2.0943951023932 effort=12 velocity=7.32666666666667 -> lower=-3.14159265358979 upper=2.0943951023932 effort=14.1 velocity=10.5; origin xyz=0.0 -0.18100293 0.23992606 rpy=0 0 0 -> xyz=0 -0.181 0.23843 rpy=0 0 0
- joint zarm_r2_joint: limit lower=-3.3161 upper=0.52 effort=12 velocity=7.32666666666667 -> lower=-3.3161 upper=0.52 effort=37.0 velocity=15.0
- joint zarm_r3_joint: limit lower=-1.5707963267949 upper=1.5707963267949 effort=12 velocity=7.32666666666667 -> lower=-1.5707963267949 upper=1.5707963267949 effort=37.0 velocity=15.0
- joint zarm_r4_joint: limit lower=-2.26892802759263 upper=0.08726 effort=12 velocity=7.32666666666667 -> lower=-2.26892802759263 upper=0.08726 effort=37.0 velocity=15.0; origin xyz=0 -0.0 -0.20533 rpy=0 0 0 -> xyz=0 0 -0.2085 rpy=0 0 0
