Commit message: sync https://www.lejuhub.com/highlydynamic/lejulab/commit/75aa852b5032d3651c64e38c54d8e97d51352095

File: src/leju_assets/models/biped_s17/urdf/drake/biped_v3_arm.urdf (robot description, URDF)
Before this commit: robot biped_v3_arm, 14 links, 13 joints
Links:
- link l_handball: geometry visual mesh filename=../../meshes/l_handball.STL
- link r_handball: geometry visual mesh filename=../../meshes/r_handball.STL
