Commit message: sync https://www.lejuhub.com/highlydynamic/lejulab/commit/4581803d496cc0b4146019305211646f62156784

File: src/leju_assets/models/biped_s54/urdf/drake/biped_v3_arm.urdf (robot description, URDF)
Before this commit: robot biped_s54, 18 links, 17 joints
Links:
- added link zarm_l7_virtual_thumb_link; collision sphere radius=0.005
- added link zarm_r7_virtual_thumb_link; collision sphere radius=0.005
Joints:
- added joint zarm_l7_virtual_thumb_joint_ee: type fixed, parent zarm_l7_end_effector, child zarm_l7_virtual_thumb_link, origin xyz=0.15 0 0 rpy=0 0 0
- added joint zarm_r7_virtual_thumb_joint_ee: type fixed, parent zarm_r7_end_effector, child zarm_r7_virtual_thumb_link, origin xyz=0.15 0 0 rpy=0 0 0
